File: DMX-ArtNET-Gateway.kicad_pcb (KiCad board)
At the start: 2 copper layers, 91.4 x 55.9 mm, 45 parts, among them J1 GPIO Breakout, J2 DMX1, J3 DMX2, J4 Barrel_Jack_MountingPin, U1 AMS1117-3.3, U2 ESP32-WROOM-32D, U3 MAX485CSA, U4 MAX485CSA

Commit message: Firmware checkin
Parts:
- added C7: 10uF, SparkFun-Capacitor:C_0805_2012Metric, F.Cu at (119.4, 94.0)
- added C8: 1uF, SparkFun-Capacitor:C_0805_2012Metric, F.Cu at (129.5, 96.5)
- added P1: USB_C_Plug_USB2.0, Connector_USB:USB_C_Receptacle_GCT_USB4105-xx-A_16P_TopMnt_Horizontal, F.Cu at (127.5, 79.5)
- added Q1: MMBT3904, Package_TO_SOT_SMD:SOT-23, F.Cu at (136.8, 132.4)
- added Q2: MMBT3904, Package_TO_SOT_SMD:SOT-23, F.Cu at (136.8, 136.8)
- added R23: 10K, SparkFun-Resistor:R_0805_2012Metric, F.Cu at (129.5, 87.6)
- added R24: 20K, SparkFun-Resistor:R_0805_2012Metric, F.Cu at (129.5, 91.4)
- added R25: 10K, SparkFun-Resistor:R_0805_2012Metric, F.Cu at (132.6, 136.8)
- added R26: 10K, SparkFun-Resistor:R_0805_2012Metric, F.Cu at (132.6, 133.0)
- added SW1: Reset, SparkFun-Switch:Momentary_SMD_4.6x2.8mm, F.Cu at (143.1, 134.2)
- added U5: CP2104, Package_DFN_QFN:QFN-24-1EP_4x4mm_P0.5mm_EP2.6x2.6mm, F.Cu at (123.8, 92.1)
- C1, C2, C5: footprint Capacitor_SMD:CP_Elec_3x5.3 -> SparkFun-Capacitor:C_0805_2012Metric
- R10: value 1k -> 10k
- moved D1 57.8 mm to (154.9, 81.3)
- moved R1 57.8 mm to (149.9, 81.3)
- moved D3 21.7 mm to (143.8, 124.5)
- moved R3 21.7 mm to (148.2, 124.5)
- moved R2 20.3 mm to (148.2, 127.0)
- moved D2 20.3 mm to (143.8, 127.0)
- moved R9 19.7 mm to (163.8, 114.3)
- moved R6 18.4 mm to (164.7, 102.9)
- moved R8 18.3 mm to (163.8, 124.5)
- moved D9 18.2 mm to (159.7, 114.3)
- moved R7 18.2 mm to (163.8, 90.2)
- moved D6 18.0 mm to (160.0, 102.9)
- moved D7 16.9 mm to (160.0, 92.7)
- moved D8 16.7 mm to (159.7, 124.5)
- moved R4 14.5 mm to (142.2, 106.7)
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Connections:
- net Net-(U2-EN) renamed CHIP_PU
- U2 pad 25: unconnected-(U2-IO0-Pad25) -> IO0
Routing:
- net +5V: track 157.8 -> 0.00 mm
- net IO21: track 89.5 -> 0.00 mm, vias 2 -> 0
- net IO2: track 70.4 -> 0.00 mm
- net IO19: track 64.2 -> 0.00 mm, vias 2 -> 0
- net IO18: track 64.1 -> 0.00 mm, vias 2 -> 0
- net IO16: track 52.1 -> 0.00 mm, vias 2 -> 0
- net IO17: track 51.7 -> 0.00 mm
- net IO23: track 50.1 -> 0.00 mm
- net DMX_2_B: track 48.3 -> 0.00 mm
- net DMX_1_B: track 48.1 -> 0.00 mm
- net IO26: track 47.3 -> 0.00 mm, vias 1 -> 0
- net IO25: track 46.5 -> 0.00 mm, vias 1 -> 0
- net IO12: track 45.3 -> 0.00 mm, vias 1 -> 0
- net IO22: track 42.9 -> 0.00 mm
- net IO14: track 42.6 -> 0.00 mm, vias 1 -> 0
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Other:
- board size 91.4 x 55.9 mm -> 91.4 x 66 mm

Commit message: Reparatie foute checkin
Parts:
- removed C7: 10uF, SparkFun-Capacitor:C_0805_2012Metric
- removed C8: 1uF, SparkFun-Capacitor:C_0805_2012Metric
- removed P1: USB_C_Plug_USB2.0, Connector_USB:USB_C_Receptacle_GCT_USB4105-xx-A_16P_TopMnt_Horizontal
- removed Q1, Q2: MMBT3904, Package_TO_SOT_SMD:SOT-23
- removed R23, R25, R26: 10K, SparkFun-Resistor:R_0805_2012Metric
- removed R24: 20K, SparkFun-Resistor:R_0805_2012Metric
- removed SW1: Reset, SparkFun-Switch:Momentary_SMD_4.6x2.8mm
- removed U5: CP2104, Package_DFN_QFN:QFN-24-1EP_4x4mm_P0.5mm_EP2.6x2.6mm
- added J5: Serial Port, Connector_PinHeader_2.54mm:PinHeader_1x04_P2.54mm_Vertical, F.Cu at (147.3, 116.8)
- R10: value 10k -> 1k
- moved R1 58.0 mm to (177.8, 132.1), turned to 0 degrees
- moved D1 54.3 mm to (174.0, 132.1), turned to 180 degrees
- moved C3 26.5 mm to (147.3, 127.0), turned to -90 degrees
- moved D3 21.7 mm to (164.2, 132.1)
- moved R3 21.7 mm to (168.5, 132.1)
- moved R2 20.3 mm to (168.5, 127.0)
- moved D2 20.3 mm to (164.1, 127.0)
- moved D9 16.2 mm to (174.0, 121.9)
- moved C2 16.1 mm to (147.3, 130.8)
- moved R9 15.9 mm to (177.8, 121.9)
- moved D6 15.3 mm to (174.0, 96.5)
- moved R4 14.5 mm to (139.7, 92.4)
- moved D8 14.5 mm to (174.0, 127.0)
- moved R5 14.5 mm to (144.8, 92.4)
- moved D4 14.5 mm to (139.7, 96.2)
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Connections:
- net CHIP_PU renamed Net-(U2-EN)
- U2 pad 25: IO0 -> unconnected-(U2-IO0-Pad25)
Routing:
- net +5V: track 0.00 -> 117.0 mm, vias 0 -> 2
- net IO18: track 0.00 -> 78.4 mm
- net IO21: track 0.00 -> 67.9 mm, vias 0 -> 2
- net IO25: track 0.00 -> 65.9 mm, vias 0 -> 1
- net IO2: track 0.00 -> 63.0 mm
- net IO19: track 0.00 -> 60.8 mm, vias 0 -> 2
- net IO26: track 0.00 -> 54.6 mm, vias 0 -> 1
- net IO16: track 0.00 -> 52.6 mm, vias 0 -> 2
- net IO17: track 0.00 -> 46.4 mm
- net IO23: track 0.00 -> 45.8 mm
- net IO14: track 0.00 -> 45.5 mm, vias 0 -> 2
- net DMX_1_B: track 0.00 -> 44.4 mm
- net IO22: track 0.00 -> 43.7 mm, vias 0 -> 1
- net RX: track 0.00 -> 43.2 mm, vias 0 -> 1
- net TX: track 0.00 -> 43.0 mm, vias 0 -> 1
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Other:
- board size 91.4 x 66 mm -> 91.4 x 55.9 mm

Commit message: Versie met TTGO-Display
Parts:
- removed C1, C2, C5: 10uF, SparkFun-Capacitor:C_0805_2012Metric
- removed C3, C4, C6: 100nF, SparkFun-Capacitor:C_0805_2012Metric
- removed J4: Barrel_Jack_MountingPin, Connector_BarrelJack:BarrelJack_CUI_PJ-102AH_Horizontal
- removed J5: Serial Port, Connector_PinHeader_2.54mm:PinHeader_1x04_P2.54mm_Vertical
- removed R10: 1k, SparkFun-Resistor:R_0805_2012Metric
- removed U1: AMS1117-3.3, Package_TO_SOT_SMD:SOT-223-3_TabPin2
- removed U2: ESP32-WROOM-32D, RF_Module:ESP32-WROOM-32D
- added TTGO1: TTGO_ESP32_TDISPLAY_V1.1, ttgo-tdisplay-kicad-master:TTGO_ESP32_TDisplay_v1.1, F.Cu at (142.2, 132.7)
- moved J1 15.2 mm to (154.9, 86.4)
- moved R12 14.3 mm to (182.9, 128.6)
- moved D4 8.75 mm to (146.1, 90.2), turned to -90 degrees
- moved D5 7.88 mm to (149.9, 90.2), turned to -90 degrees
- moved R4 6.97 mm to (146.1, 95.2), turned to 90 degrees
- moved R5 5.84 mm to (149.9, 95.2), turned to 90 degrees
- moved R20 1.21 mm to (154.0, 115.5)
- moved R21 1.21 mm to (154.0, 118.0)
- moved R22 1.21 mm to (154.0, 120.5)
- moved U4 1.20 mm to (161.2, 118.0)
- moved R17 0.91 mm to (153.7, 102.2)
- moved R18 0.91 mm to (153.7, 99.7)
- moved R19 0.91 mm to (153.7, 97.2)
- moved U3 0.91 mm to (160.9, 99.7)
Connections:
- net IO19 renamed IO27
- D7 pad 1: IO16 -> IO15
- D9 pad 1: IO18 -> IO22
- J1 pad 1: IO5 -> IO2
- J1 pad 10: IO26 -> +3.3V
- J1 pad 3: IO13 -> IO21
- J1 pad 4: IO14 -> IO32
- J1 pad 5: IO15 -> IO33
- J1 pad 6: IO21 -> IO37
- J1 pad 7: IO22 -> IO38
- J1 pad 8: IO23 -> TX
- J1 pad 9: IO25 -> RX
- R18 pad 2: IO4 -> IO12
- R19 pad 2: IO16 -> IO15
- R20 pad 2: IO18 -> IO22
- U3 pad 1: IO16 -> IO15
- U3 pad 2: IO4 -> IO12
- U3 pad 3: IO4 -> IO12
- U4 pad 1: IO18 -> IO22
Routing:
- net IO18: track 78.4 -> 0.00 mm
- net IO25: track 65.9 -> 0.00 mm, vias 1 -> 0
- net IO2: track 63.0 -> 126.4 mm
- net IO26: track 54.6 -> 0.00 mm, vias 1 -> 0
- net IO16: track 52.6 -> 0.00 mm, vias 2 -> 0
- net IO23: track 45.8 -> 0.00 mm
- net IO14: track 45.5 -> 0.00 mm, vias 2 -> 0
- net IO38: track 0.00 -> 35.0 mm
- net IO13: track 33.9 -> 0.00 mm, vias 1 -> 0
- net RX: track 43.2 -> 75.8 mm
- net IO33: track 0.00 -> 31.5 mm
- net IO37: track 0.00 -> 30.1 mm
- net IO15: track 32.2 -> 61.4 mm, vias 1 -> 0
- net IO32: track 0.00 -> 28.2 mm
- net IO12: track 37.2 -> 64.6 mm, vias 1 -> 3
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