File: DMX-ArtNET-Gateway.kicad_sch (KiCad schematic)
At the start: 45 parts, among them J1 GPIO Breakout, J2 DMX1, J3 DMX2, J4 Barrel_Jack_MountingPin, U1 AMS1117-3.3, U2 ESP32-WROOM-32D, U3 MAX485CSA, U4 MAX485CSA

Commit message: Firmware checkin
Parts:
- added C7: 10uF, Capacitor_SMD:CP_Elec_3x5.3, symbol SparkFun-Capacitor:10uF_0603_6.3V_20%
- added C8: 1uF, Capacitor_SMD:CP_Elec_3x5.3, symbol SparkFun-Capacitor:10uF_0603_6.3V_20%
- added P1: USB_C_Plug_USB2.0, Connector_USB:USB_C_Receptacle_GCT_USB4105-xx-A_16P_TopMnt_Horizontal, symbol Connector:USB_C_Plug_USB2.0
- added Q1, Q2: MMBT3904, Package_TO_SOT_SMD:SOT-23, symbol Transistor_BJT:MMBT3904
- added R23, R25, R26: 10K, SparkFun-Resistor:R_0805_2012Metric, symbol SparkFun-Resistor:R
- added R24: 20K, SparkFun-Resistor:R_0805_2012Metric, symbol SparkFun-Resistor:R
- added SW1: Reset, SparkFun-Switch:Momentary_SMD_4.6x2.8mm, symbol SparkFun-Switch:SPST_Momentary_4.6x2.8mm
- added U5: CP2104, Package_DFN_QFN:QFN-24-1EP_4x4mm_P0.5mm_EP2.6x2.6mm, symbol Interface_USB:CP2104
- R10: value 1k -> 10k
Connections:
- net +3.3V: now also C8.1, U5.5 (VIO), U5.6 (VDD), U5.7 (REGIN)
- net +5V: now also P1.A4 (VBUS), P1.A9 (VBUS), P1.B4 (VBUS), P1.B9 (VBUS), R23.1
- net GND: now also C7.2, C8.2, P1.A1 (GND), P1.A12 (GND), P1.B1 (GND), P1.B12 (GND), P1.S1 (SHIELD), R24.1, SW1.1 (A), U5.2 (GND), U5.25 (GND)
- net RX: now also U5.21 (TXD)
- net TX: now also U5.20 (RXD)
- net CHIP_PU: now reaches C6.1, R10.2, U2.3 (EN)
- net CHIP_PU: now also Q1.3 (C), SW1.2 (B)
- net IO0: now reaches U2.25 (IO0)
- net IO0: now also Q2.3 (C)
- new net: Q1.1 (B), R25.1
- new net: C7.1, U5.16 (VPP)
- new net: Q2.1 (B), R26.1
- new net D+: P1.A6 (D+), U5.3 (D+)
- new net D-: P1.A7 (D-), U5.4 (D-)
- new net DTR: Q2.2 (E), R25.2, U5.23 (~{DTR})
- new net RTS: Q1.2 (E), R26.2, U5.19 (~{RTS})
- new net VBUS: R23.2, R24.2, U5.8 (VBUS)
- no-connect marks 14 -> 26
Other:
- moved on the sheet: C5, C6, J1, J2, J3, R10, R11, R12, R13, R14, R15, R16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

Commit message: Reparatie foute checkin
Parts:
- removed C7: 10uF, Capacitor_SMD:CP_Elec_3x5.3, symbol SparkFun-Capacitor:10uF_0603_6.3V_20%
- removed C8: 1uF, Capacitor_SMD:CP_Elec_3x5.3, symbol SparkFun-Capacitor:10uF_0603_6.3V_20%
- removed P1: USB_C_Plug_USB2.0, Connector_USB:USB_C_Receptacle_GCT_USB4105-xx-A_16P_TopMnt_Horizontal, symbol Connector:USB_C_Plug_USB2.0
- removed Q1, Q2: MMBT3904, Package_TO_SOT_SMD:SOT-23, symbol Transistor_BJT:MMBT3904
- removed R23, R25, R26: 10K, SparkFun-Resistor:R_0805_2012Metric, symbol SparkFun-Resistor:R
- removed R24: 20K, SparkFun-Resistor:R_0805_2012Metric, symbol SparkFun-Resistor:R
- removed SW1: Reset, SparkFun-Switch:Momentary_SMD_4.6x2.8mm, symbol SparkFun-Switch:SPST_Momentary_4.6x2.8mm
- removed U5: CP2104, Package_DFN_QFN:QFN-24-1EP_4x4mm_P0.5mm_EP2.6x2.6mm, symbol Interface_USB:CP2104
- added J5: Serial Port, Connector_PinHeader_2.54mm:PinHeader_1x04_P2.54mm_Vertical, symbol Connector:Conn_01x04_Pin
- C1, C2, C5: footprint Capacitor_SMD:CP_Elec_3x5.3 -> SparkFun-Capacitor:C_0805_2012Metric
- R10: value 10k -> 1k
Connections:
- net +5V: now also J5.1 (Pin_1)
- net GND: now also J5.4 (Pin_4); no longer J4.MP (MountPin)
- net RX: now also J5.3 (Pin_3)
- net TX: now also J5.2 (Pin_2)
- net CHIP_PU: no longer names the net of C6.1, R10.2, U2.3 (EN)
- net IO0: no longer names the net of U2.25 (IO0)
- no-connect marks 26 -> 17
Other:
- moved on the sheet: C5, C6, J1, J2, J3, R10, R11, R12, R13, R14, R15, R16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

Commit message: Versie met TTGO-Display
Parts:
- removed C1, C2, C5: 10uF, SparkFun-Capacitor:C_0805_2012Metric, symbol SparkFun-Capacitor:10uF_0603_6.3V_20%
- removed C3, C4, C6: 100nF, SparkFun-Capacitor:C_0805_2012Metric, symbol SparkFun-Capacitor:C
- removed J4: Barrel_Jack_MountingPin, Connector_BarrelJack:BarrelJack_CUI_PJ-102AH_Horizontal, symbol Connector:Barrel_Jack_MountingPin
- removed J5: Serial Port, Connector_PinHeader_2.54mm:PinHeader_1x04_P2.54mm_Vertical, symbol Connector:Conn_01x04_Pin
- removed R10: 1k, SparkFun-Resistor:R_0805_2012Metric, symbol SparkFun-Resistor:R
- removed U1: AMS1117-3.3, Package_TO_SOT_SMD:SOT-223-3_TabPin2, symbol Regulator_Linear:AMS1117-3.3
- removed U2: ESP32-WROOM-32D, RF_Module:ESP32-WROOM-32D, symbol RF_Module:ESP32-WROOM-32D
- added TTGO1: TTGO_ESP32_TDISPLAY_V1.1, ttgo-tdisplay-kicad-master:TTGO_ESP32_TDisplay_v1.1, symbol ttgo_esp32:TTGO_ESP32_TDISPLAY_V1.1
Connections:
- net IO16 is gone; now on net IO15: D7.1 (K), R19.2, U3.1 (RO)
- net IO18 is gone; now on net IO22: D9.1 (K), R20.2, U4.1 (RO)
- net IO23 is gone; now on net TX: J1.8 (Pin_8)
- net IO25 is gone; now on net RX: J1.9 (Pin_9)
- net IO26 is gone; now on net +3.3V: J1.10 (Pin_10)
- net IO4 is gone; now on net IO12: R18.2, U3.2 (~{RE}), U3.3 (DE)
- net IO5 is gone; now on net IO2: J1.1 (Pin_1)
- net +3.3V: now also TTGO1.12 (3.3V), TTGO1.24 (3.3V)
- net +5V: now also TTGO1.1 (5V)
- net GND: now also TTGO1.13 (GND), TTGO1.14 (GND), TTGO1.2 (GND), TTGO1.22 (GND), TTGO1.23 (GND)
- net IO12: now also TTGO1.21 (GPIO12)
- net IO13: now also TTGO1.20 (GPIO13); no longer J1.3 (Pin_3)
- net IO15: now also TTGO1.19 (GPIO15); no longer J1.5 (Pin_5)
- net IO17: now also TTGO1.17 (GPIO17)
- net IO2: now also TTGO1.18 (GPIO2)
- net IO21: now also J1.3 (Pin_3), TTGO1.15 (GPIO21); no longer J1.6 (Pin_6)
- net IO22: now also TTGO1.16 (GPIO22); no longer J1.7 (Pin_7)
- net RX: now also TTGO1.4 (GPIO26)
- net TX: now also TTGO1.5 (GPIO25)
- net IO14 renamed IO32
- net IO32: now also TTGO1.7 (GPIO32)
- net IO19 renamed IO27
- net IO27: now also TTGO1.3 (GPIO27)
- new net IO33: J1.5 (Pin_5), TTGO1.6 (GPIO33)
- new net IO37: J1.6 (Pin_6), TTGO1.10 (GPIO37)
- new net IO38: J1.7 (Pin_7), TTGO1.9 (GPIO38)
- no-connect marks 17 -> 2
